Commit message: Actualizacion del bot y el mundo

File: src/puzzlebot_gazebo/urdf/parameters.xacro (robot description, xacro)
@@ -22,3 +22,4 @@
 <xacro:property name="mesh_wheel"  value="$(find puzzlebot_gazebo)/meshes/wheel.stl" />
 <xacro:property name="mesh_camera"  value="$(find puzzlebot_gazebo)/meshes/camera.stl" />
+<xacro:property name="mesh_lidar"  value="$(find puzzlebot_gazebo)/meshes/lidar.stl" />
 </robot>

File: src/puzzlebot_gazebo/urdf/puzzlebot_mod.xacro (robot description, xacro)
@@ -135,4 +135,54 @@
         </visual>
     </link>
+		<!-- LIDAR-->
+	<link name="$(arg prefix)lidar">
+		<inertial>
+			<mass value="0.1" />
+			<origin xyz="0 0 0" />
+			<inertia ixx="0.01" ixy="0.0" ixz="0.0"
+					 iyy="0.01" iyz="0.0"
+					 izz="0.01" />
+		</inertial>
+		<!-- <visual>
+			<origin xyz=" 0 0 0 " rpy="0 0 0" />
+			<geometry>
+				<cylinder length="0.05" radius="0.05"/>
+			</geometry>
+			<material name="black"/>
+		</visual> -->
+		<collision>
+			<origin xyz="-0.06 0.0 -0.04" rpy="0 0 0" />
+			<geometry>
+				<cylinder length="0.01" radius="0.05"/>
+			</geometry>
+		</collision>
+        <visual>
+			<origin rpy="${PI/2} 0 0" xyz="0.07 -0.013 -0.04" />
+            <geometry>
+                <mesh filename="file://${mesh_lidar}" />
+            </geometry>
+        </visual>
+		<![CDATA[
+        <collision>
+			<origin rpy="0 0 0" xyz="0 0 0" />
+			<!-- <geometry>
+				<box size="1000 1000 0.01" />
+			</geometry> -->
+			<geometry>
+				<!-- <mesh filename="file://${mesh_lidar}" /> -->
+				<!-- <box size="0.01 0.01 0.01" /> -->
+				<cylinder length="0.01" radius="0.5" />
+			</geometry>
+        </collision>
+        <!-- <inertial_cylinder mass="0.1" length="0.04" radius="0.05">
+            <origin xyz="0 0 0" rpy="0 0 0"/>
+        </inertial_cylinder> -->
+		<inertial>
+			<origin rpy="0 0 0" xyz="0 0 0" />
+			<mass value="0.000" />
+			<inertia ixx="0.166667" ixy="0" ixz="0" iyy="0.166667" iyz="0" izz="0.166667" />
+			<!-- ad camera inertia -->
+		</inertial>]]>
+    </link>
 <!-- JOINTS  -->
   <joint name="base_to_right_w" type="continuous">
@@ -158,4 +208,9 @@
 		<origin xyz="0.09 0 0.048" rpy= "0.0 0.24 0.0" />
   	</joint>
+	<joint name="lidar_to_base" type="fixed">
+        <parent link="$(arg prefix)chassis"/>
+        <child link="$(arg prefix)lidar"/>
+        <origin xyz="0.05 0 0.115" rpy="0 0 ${PI}"/>
+    </joint>
 	<!-- TRANSMISSIONS (For a more complex model and it represents actuator attributes) -->
 	<transmission name="right_wheel_trans">
