Commit message: Aruco detection completed

File: src/puzzlebot_gazebo/urdf/puzzlebot_mod.xacro (robot description, xacro)
@@ -129,5 +129,5 @@
                 </geometry>-->
                 <!-- with mesh-->
-                <origin rpy="${PI/2} 0 ${PI/2}" xyz="0 0 0"/>
+                <origin rpy="0 0 ${PI}" xyz="0 0 0"/>
                 <geometry>
                 <mesh filename="file://${mesh_camera}"/>
@@ -144,11 +144,4 @@
 					 izz="0.01" />
 		</inertial>
-		<!-- <visual>
-			<origin xyz=" 0 0 0 " rpy="0 0 0" />
-			<geometry>
-				<cylinder length="0.05" radius="0.05"/>
-			</geometry>
-			<material name="black"/>
-		</visual> -->
 		<collision>
 			<origin xyz="-0.06 0.0 -0.04" rpy="0 0 0" />
@@ -163,25 +156,4 @@
             </geometry>
         </visual>
-		<![CDATA[
-        <collision>
-			<origin rpy="0 0 0" xyz="0 0 0" />
-			<!-- <geometry>
-				<box size="1000 1000 0.01" />
-			</geometry> -->
-			<geometry>
-				<!-- <mesh filename="file://${mesh_lidar}" /> -->
-				<!-- <box size="0.01 0.01 0.01" /> -->
-				<cylinder length="0.01" radius="0.5" />
-			</geometry>
-        </collision>
-        <!-- <inertial_cylinder mass="0.1" length="0.04" radius="0.05">
-            <origin xyz="0 0 0" rpy="0 0 0"/>
-        </inertial_cylinder> -->
-		<inertial>
-			<origin rpy="0 0 0" xyz="0 0 0" />
-			<mass value="0.000" />
-			<inertia ixx="0.166667" ixy="0" ixz="0" iyy="0.166667" iyz="0" izz="0.166667" />
-			<!-- ad camera inertia -->
-		</inertial>]]>
     </link>
 <!-- JOINTS  -->
@@ -206,5 +178,6 @@
 		<parent link="$(arg prefix)chassis" />
 		<child link="$(arg prefix)camera" />
-		<origin xyz="0.09 0 0.048" rpy= "0.0 0.24 0.0" />
+		<origin xyz="0.09 0 0.048" rpy= "${PI/2} ${PI} ${PI/2}" />
+		<!-- <origin xyz="0.09 0 0.048" rpy= "0.0 0.0 0.0" /> -->
   	</joint>
 	<joint name="lidar_to_base" type="fixed">
